File: modulo_arduino/pcb_mod_arduino.sch (KiCad schematic (older format))
At the start: 8 parts, among them J1 modulo 1, J2 modulo 2, J3 modulo 3, J4 modulo 4, J5 modulo 5, J6 modulo 6, J7 power

Commit message: marcas pines, reemplazo borneras, orientacion, separacion headers, ubicacion arduino
Parts:
- J7: footprint Pin_Headers:Pin_Header_Straight_1x04_Pitch2.54mm -> Connectors_Terminal_Blocks:TerminalBlock_bornier-4_P5.08mm
Connections:
- net +5V: now also XA1.VIN
- no-connect marks 43 -> 42
Changed lines of the file:
@@
 LIBS:valves
 LIBS:arduino
+LIBS:pcb_mod_arduino-cache
 EELAYER 25 0
 EELAYER END
@@
 F 0 "J7" H 7650 1300 50  0000 C CNN
 F 1 "power" H 7650 800 50  0000 C CNN
-F 2 "Pin_Headers:Pin_Header_Straight_1x04_Pitch2.54mm" H 7650 1100 50  0001 C CNN
+F 2 "Connectors_Terminal_Blocks:TerminalBlock_bornier-4_P5.08mm" H 7650 1100 50  0001 C CNN
 F 3 "" H 7650 1100 50  0001 C CNN
 	1    7650 1100
@@
 NoConn ~ 1750 5950
 NoConn ~ 1750 6050
-NoConn ~ 1750 6150
 NoConn ~ 2800 1400
 NoConn ~ 2900 1400
@@
 Wire Wire Line
 	3200 1300 3200 1400
+Text Label 1500 6150 2    60   ~ 0
+vin
+Wire Wire Line
+	1500 6150 1750 6150
+Text Label 7950 1400 0    60   ~ 0
+vin
+Wire Wire Line
+	7950 1400 7850 1400
+Connection ~ 7850 1400
 $EndSCHEMATC
