File: modulo_botones/pcb_mod_btn.sch (KiCad schematic (older format))
At the start: 51 parts, among them J1 leds_1, J10 leds_2, J11 led_3, J12 btn_3, J13 leds_4, J14 leds_4, J15 leds_4, J16 leds_4, J17 btn_4, J18 leds_5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

Commit message: marcas pines, reemplazo borneras, orientacion, separacion headers, ubicacion arduino
Parts:
- J25: footprint Pin_Headers:Pin_Header_Straight_1x04_Pitch2.54mm -> Connectors_Terminal_Blocks:TerminalBlock_bornier-4_P5.08mm
Changed lines of the file:
@@
 F 0 "J25" H 7900 4300 50  0000 C CNN
 F 1 "power" H 7900 3800 50  0000 C CNN
-F 2 "Pin_Headers:Pin_Header_Straight_1x04_Pitch2.54mm" H 7900 4100 50  0001 C CNN
+F 2 "Connectors_Terminal_Blocks:TerminalBlock_bornier-4_P5.08mm" H 7900 4100 50  0001 C CNN
 F 3 "" H 7900 4100 50  0001 C CNN
 	1    7900 4100
